File: Robot-Arm-Breakout/Robot-Arm-Breakout.kicad_sch (KiCad schematic)
At the start: 7 parts, among them J1 Pico-Parrallel, J2 Conn_01x03_Pin, J3 Conn_01x03_Pin, J4 Conn_01x03_Pin, J5 Conn_01x03_Socket, J6 Conn_01x03_Socket, J7 Conn_01x03_Socket

Commit message: Commit before Combining boards with mousebites
Parts:
- added H1, H2, H3: MountingHole, MountingHole:MountingHole_3.2mm_M3, symbol Mechanical:MountingHole
- added J10, J8, J9: Conn_01x03_Pin, Connector_PinHeader_2.54mm:PinHeader_1x03_P2.54mm_Horizontal, symbol Connector:Conn_01x03_Pin
- added RV1, RV2, RV3: R_Potentiometer_US, Footprints-General:Potentiometer-Multi, symbol Device:R_Potentiometer_US
- J5, J6, J7: footprint (none) -> Connector_PinSocket_2.54mm:PinSocket_1x03_P2.54mm_Vertical
Connections:
- net ADC0: now also J5.3 (Pin_3); no longer J5.1 (Pin_1)
- net ADC1: now also J6.3 (Pin_3); no longer J6.1 (Pin_1)
- net ADC2: now also J7.3 (Pin_3); no longer J7.1 (Pin_1)
- net GND: now also J1.13 (Pin_13), J5.1 (Pin_1), J6.1 (Pin_1), J7.1 (Pin_1); no longer J5.3 (Pin_3), J6.3 (Pin_3), J7.3 (Pin_3)
- new net Pot_Board1_3v3: J8.2 (Pin_2), RV1.1
- new net Pot_Board1_GND: J8.1 (Pin_1), RV1.3
- new net Pot_Board1_Sense: J8.3 (Pin_3), RV1.2
- new net Pot_Board2_3v3: J9.2 (Pin_2), RV2.1
- new net Pot_Board2_GND: J9.1 (Pin_1), RV2.3
- new net Pot_Board2_Sense: J9.3 (Pin_3), RV2.2
- new net Pot_Board3_3v3: J10.2 (Pin_2), RV3.1
- new net Pot_Board3_GND: J10.1 (Pin_1), RV3.3
- new net Pot_Board3_Sense: J10.3 (Pin_3), RV3.2
- no-connect marks 6 -> 5
Other:
- note added: "GND"
- note added: "Pico"
- note added: "Potentiometer Boards"
- note added: "Potentiometer connectors"
- note added: "Servo Connectors"
- company: (none) -> Liam Howell
- title: (none) -> Robot Arm Pico Wing
- moved on the sheet: J1, J2, J3, J4, J5, J6, J7
